File: project_A.kicad_sch (KiCad schematic)
At the start: 1 part

Commit message: add .svg - test --test
Connections:
- net dddd renamed aaaa
Changed lines of the file:
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@@
     (stroke (width 0) (type default) (color 0 0 0 0))
   )
-  (global_label "dddd" (shape input) (at 204.47 43.18 0) (fields_autoplaced)
+  (global_label "aaaa" (shape input) (at 204.47 43.18 0) (fields_autoplaced)
     (effects (font (size 1.27 1.27)) (justify left))
     (property "Intersheet References" "${INTERSHEET_REFS}" (id 0) (at 211.4793 43.1006 0)

Commit message: feat : 기능추가
Signed-off-by: NOHsi <lws20820@greenlabs.co.kr>
Parts:
- added 24+H1, 24+H2: MountingHole, Connector_Pin:Pin_D1.3mm_L11.3mm_W2.8mm_Flat, symbol Mechanical:MountingHole
- added BT1: Battery_Cell, Battery:BatteryHolder_Keystone_1058_1x2032, symbol Device:Battery_Cell
- added C1, C2: C104, Capacitor_SMD:C_1206_3216Metric, symbol Device:C
- added C3: 10uF/50V(C3216), Capacitor_SMD:CP_Elec_6.3x4.5, symbol Device:C_Polarized_US
- added C4, C5, C6: C104, Capacitor_SMD:C_0805_2012Metric_Pad1.18x1.45mm_HandSolder, symbol Device:C
- added C7: 100uF/50V, Capacitor_SMD:CP_Elec_6.3x4.5, symbol Device:C_Polarized_US
- added CN1: Conn_01x04, Connector:FanPinHeader_1x04_P2.54mm_Vertical, symbol Connector_Generic:Conn_01x04
- added CN2: Conn_01x04, Connector_IDC:IDC-Header_2x03_P2.54mm_Horizontal, symbol Connector_Generic:Conn_01x04
- added D1: STPS3L60U, Diode_SMD:D_SMB, symbol pspice:DIODE
- added J1: SD_Card, Connector_Card:microSD_HC_Hirose_DM3D-SF, symbol Connector:SD_Card
- added L1: 10uH(YCDM6045T), Inductor_SMD:L_7.3x7.3_H4.5, symbol Device:L
- added R1: 47K(R1608), Resistor_SMD:R_0805_2012Metric_Pad1.20x1.40mm_HandSolder, symbol Device:R_US
- added R2, R3: 187K(R1608), Resistor_SMD:R_0805_2012Metric_Pad1.20x1.40mm_HandSolder, symbol Device:R_US
- added R4, R5: 1K, Resistor_SMD:R_0805_2012Metric_Pad1.20x1.40mm_HandSolder, symbol Device:R_US
- added U1: LT1129-3.3_SOT223, Package_TO_SOT_SMD:SOT-223-3_TabPin2, symbol Regulator_Linear:LT1129-3.3_SOT223
- added U2: ST1S14PHR, Package_SO:TI_SO-PowerPAD-8, symbol Regulator_Switching:ST1S14PHR
- added U4: DS3231M, Package_SO:SOIC-16W_7.5x10.3mm_P1.27mm, symbol Timer_RTC:DS3231M
- gave numbers to parts that had none: 1
Connections:
- net GND: now also C1.2, C2.2, C3.2, C4.2, C7.2, CN1.2 (Pin_2), D1.1 (K), R3.1, U1.2 (GND), U2.6 (GND), U2.9 (PADGND)
- net SDA: now reaches U3.8 (IO32)
- net SDA: now also R5.1, U4.15 (SDA)
- net SCL: now reaches U3.9 (IO33)
- net SCL: now also R4.1, U4.16 (SCL)
- net +3.3VDAC renamed +3.3V
- net +3.3V: now also C2.1, R4.2, R5.2, U1.3 (VO)
- new net: U4.10 (GND), U4.11 (GND), U4.12 (GND), U4.13 (GND), U4.5 (GND), U4.6 (GND), U4.7 (GND), U4.8 (GND), U4.9 (GND)
- new net: R1.1, U2.2 (PG)
- new net: C6.2, R1.2, R2.2
- new net: C6.1, R2.1, R3.2, U2.4 (FB)
- new net: C5.1, U2.1 (BOOT)
- new net: C5.2, D1.2 (A), L1.1, U2.8 (SW)
- new net +24V: C3.1, C4.1, U2.5 (EN2), U2.7 (VIN)
- new net +5V: C1.1, CN1.1 (Pin_1), U1.1 (VI)
- new net +5V OUT: C7.1, L1.2
- new net rx: CN1.3 (Pin_3)
- new net tx: CN1.4 (Pin_4)
